File: Board_Files/DEC_R_BOX.kicad_pcb (KiCad board)
At the start: 2 copper layers, 75 x 131.6 mm, 86 parts, among them J1 Conn_01x01_Socket, J2 Conn_01x01_Socket, SW1 SW_SPDT, SW10 SW_SPDT, SW11 SW_SPDT, SW12 SW_SPDT, SW13 SW_SPDT, SW14 SW_SPDT, SW15 SW_SPDT, SW16 SW_SPDT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

Commit message: Iniital Commit
Other:
- board text added: "DECADE RESISTANCE BOARD : 1Ω - 1MEGAΩ"
- board text removed: "DECADE RESISTANC BOARD : 1Ω - 1MEGAΩ"
